Commit message: first commit

File: arduino_bot_desc/urdf/arduinobot.urdf.xacro (robot description, xacro)
@@ -1,8 +1,27 @@
 <?xml version="1.0"?>
-<robot xmlns:xacro="http://www.ros.org/wiki/xacro" name="robot_name">
+<robot xmlns:xacro="http://www.ros.org/wiki/xacro" name="arduino_bot">
+    <xacro:include filename="$(find arduino_bot_desc)/urdf/arduinobot_ros2_control.xacro"/>
+    <xacro:include filename="$(find arduino_bot_desc)/urdf/arduinobot_gazebo.xacro"/>
     <xacro:property name="PI" value="3.14159" />
     <xacro:property name="effort" value="30.0" />
     <xacro:property name="velocity" value="10.0" />
     <xacro:property name="stl_path" value="package://arduino_bot_desc/meshes/" />
+    <xacro:macro name="default_inertial" params="mass">
+        <inertial>
+            <origin xyz="0.0 0.0 0.0" rpy="0.0 0.0 0.0"/>
+            <mass value="${mass}"/>
+            <inertia ixx="1.0" ixy="0.0" ixz="0.0" iyy="1.0" iyz="0.0" izz="1.0"/>
+        </inertial>
+    </xacro:macro>
+    <xacro:macro name="default_transmission" params="number">
+        <transmission name="trans_${number}">
+            <plugin>transmission_interface/SimpleTransmission</plugin>
+            <joint name="joint_${number}">
+                <mechanical_reduction>1.0</mechanical_reduction>
+                <hardwareInterface>hardware_interface/PositionJointInterface</hardwareInterface>
+            </joint>
+            <actuator name="motor_${number}" role="actuator1"/>
+        </transmission>
+    </xacro:macro>
     <link name="world"/>
     <link name="base_link">
@@ -13,4 +32,11 @@
             </geometry>
         </visual>
+        <collision>
+            <origin xyz="-0.5 -0.5 0" rpy="0 0 0"/>
+            <geometry>
+                <mesh filename="${stl_path}basement.STL" scale="0.01 0.01 0.01"/>
+            </geometry>
+        </collision>
+        <xacro:default_inertial mass="1.0"/>
     </link>
     <joint name="my_virtual_joint" type="fixed">
@@ -26,4 +52,11 @@
             </geometry>
         </visual>
+        <collision>
+            <origin xyz="-0.39 -0.39 -0.56" rpy="0.0 0.0 0.0"/>
+            <geometry>
+                <mesh filename="${stl_path}base_plate.STL" scale="0.01 0.01 0.01"/>
+            </geometry>
+        </collision>
+        <xacro:default_inertial mass="0.1"/>
     </link>
     <joint name="joint_1" type="revolute">
@@ -41,4 +74,11 @@
             </geometry>
         </visual>
+        <collision>
+            <origin xyz="0.19 0.06 -0.08" rpy="0.0 -${PI/2} ${PI/2}"/>
+            <geometry>
+                <mesh filename="${stl_path}forward_drive_arm.STL" scale="0.01 0.01 0.01"/>
+            </geometry>
+        </collision>
+        <xacro:default_inertial mass="0.1"/>
     </link>
     <joint name="joint_2" type="revolute">
@@ -56,4 +96,11 @@
             </geometry>
         </visual>
+        <collision>
+            <origin xyz="-0.03 -0.4 -0.06" rpy="${PI/2} 0 ${PI/2}"/>
+            <geometry>
+                <mesh filename="${stl_path}horizontal_arm.STL" scale="0.01 0.01 0.01"/>
+            </geometry>
+        </collision>
+        <xacro:default_inertial mass="0.1"/>
     </link>
     <joint name="joint_3" type="revolute">
@@ -71,4 +118,11 @@
             </geometry>
         </visual>
+        <collision>
+            <origin xyz="0 -0.05 -0.15" rpy="0 0 ${PI/2}"/>
+            <geometry>
+                <mesh filename="${stl_path}claw_support.STL" scale="0.01 0.01 0.01"/>
+            </geometry>
+        </collision>
+        <xacro:default_inertial mass="0.05"/>
     </link>
     <joint name="horizontal_arm_to_claw_support" type="fixed">
@@ -84,4 +138,11 @@
             </geometry>
         </visual>
+        <collision>
+            <origin xyz="-0.1 0.5 -0.1" rpy="0 0 -${PI/2}"/>
+            <geometry>
+                <mesh filename="${stl_path}right_finger.STL" scale="0.01 0.01 0.01"/>
+            </geometry>
+        </collision>
+        <xacro:default_inertial mass="0.05"/>
     </link>
     <link name="gripper_left">
@@ -92,4 +153,11 @@
             </geometry>
         </visual>
+        <collision>
+            <origin xyz="-0.04 0.5 -0.1" rpy="0 0 -${PI/2}"/>
+            <geometry>
+                <mesh filename="${stl_path}left_finger.STL" scale="0.01 0.01 0.01"/>
+            </geometry>
+        </collision>
+        <xacro:default_inertial mass="0.05"/>
     </link>
     <joint name="joint_4" type="revolute">
@@ -108,3 +176,7 @@
         <mimic joint="joint_4" multiplier="-1"/>
     </joint>
+    <xacro:default_transmission number="1"/>
+    <xacro:default_transmission number="2"/>
+    <xacro:default_transmission number="3"/>
+    <xacro:default_transmission number="4"/>
 </robot>

Commit message: class finished. bug fixes remaining

File: arduino_bot_desc/urdf/arduinobot.urdf.xacro (robot description, xacro)
@@ -1,4 +1,5 @@
 <?xml version="1.0"?>
 <robot xmlns:xacro="http://www.ros.org/wiki/xacro" name="arduinobot">
+    <xacro:arg name="is_sim" default="true"/>
     <xacro:include filename="$(find arduino_bot_desc)/urdf/arduinobot_ros2_control.xacro"/>
     <xacro:include filename="$(find arduino_bot_desc)/urdf/arduinobot_gazebo.xacro"/>

File: arduino_bot_desc/urdf/arduinobot_ros2_control.xacro (robot description, xacro)
@@ -1,9 +1,26 @@
 <?xml version="1.0"?>
 <robot xmlns:xacro="http://www.ros.org/wiki/xacro">
-    <xacro:property name="PI" value="3.14159" />
     <ros2_control name="RobotSystem" type="system">
-        <hardware>
-            <plugin>gazebo_ros2_control/GazeboSystem</plugin>
-        </hardware>
+        <xacro:property name="PI" value="3.14159" />
+        <xacro:if value="$(arg is_sim)">
+            <hardware>
+                <plugin>gazebo_ros2_control/GazeboSystem</plugin>
+            </hardware>
+            <joint name="joint_5">
+                <command_interface name = "position">
+                    <param name = "min">0</param>
+                    <param name = "max">${PI/2}</param>
+                </command_interface>
+                <state_interface name = "position"/>
+                <mimic joint = "joint_4" multiplier = "-1"/>
+            </joint>
+        </xacro:if>
+        <xacro:unless value="$(arg is_sim)">
+            <hardware>
+                <plugin>arduino_bot_controller/ArduinobotInterface</plugin>
+                <param name="port">/dev/ttyACM0</param>
+            </hardware>
+        </xacro:unless>
+        <xacro:property name="PI" value="3.14159" />
         <joint name="joint_1">
             <command_interface name = "position">
@@ -34,12 +51,4 @@
             <state_interface name = "position"/>
         </joint>
-        <joint name="joint_5">
-            <command_interface name = "position">
-                <param name = "min">0</param>
-                <param name = "max">${PI/2}</param>
-            </command_interface>
-            <state_interface name = "position"/>
-            <mimic joint = "joint_4" multiplier = "-1"/>
-        </joint>
     </ros2_control>
 </robot>
