Commit message: fixed gripper mimic bug.

File: arduino_bot_desc/urdf/arduinobot_ros2_control.xacro (robot description, xacro)
@@ -8,4 +8,6 @@
             </hardware>
             <joint name="joint_5">
+                <param name="mimic">joint_4</param>
+                <param name="multiplier">-1</param>
                 <command_interface name = "position">
                     <param name = "min">0</param>
@@ -13,5 +15,5 @@
                 </command_interface>
                 <state_interface name = "position"/>
-                <mimic joint = "joint_4" multiplier = "-1"/>
+                <!-- <mimic joint = "joint_4" multiplier = "-1"/> -->
             </joint>
         </xacro:if>

Commit message: real robot not working

File: arduino_bot_desc/urdf/arduinobot_ros2_control.xacro (robot description, xacro)
@@ -8,6 +8,6 @@
             </hardware>
             <joint name="joint_5">
-                <param name="mimic">joint_4</param>
-                <param name="multiplier">-1</param>
+                <!-- <param name="mimic">joint_4</param>
+                <param name="multiplier">-1</param> -->
                 <command_interface name = "position">
                     <param name = "min">0</param>
@@ -15,5 +15,5 @@
                 </command_interface>
                 <state_interface name = "position"/>
-                <!-- <mimic joint = "joint_4" multiplier = "-1"/> -->
+                <mimic joint = "joint_4" multiplier = "-1"/>
             </joint>
         </xacro:if>
